File: DC_driver/DC_driver.sch (KiCad schematic (older format))
At the start: 38 parts, among them J1 CONN_01X10, J2 CONN_01X10, J3 CONN_01X10, J4 CONN_01X10, P1 CONN_01X02, P2 CONN_01X02, U1 MC34063A, U2 NTD3055L104-D, U3 NTD3055L104-D, U4 NTD3055L104-D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

Commit message: main changes
Parts:
- removed C10, C9: 470 uF, Capacitors_ThroughHole:C_Radial_D10_L21_P5, symbol CP
- removed C2: C, Capacitors_SMD:C_1206, symbol C
- removed D1: D_Schottky, Diodes_SMD:9.40x3.30, symbol D_Schottky
- removed JP1: JUMPER, Pin_Headers:Pin_Header_Straight_1x02, symbol JUMPER
- removed L1: L_Small, Inductors:SELF-WE-PD-XXL, symbol L_Small
- removed R1: R, Resistors_SMD:R_1206, symbol R
- removed RV1: POT, Potentiometers:Potentiometer_Bourns_3296Y_3-8Zoll_Angular_ScrewUp, symbol POT
- removed U1: MC34063A, Housings_SOIC:SOIC-8_3.9x4.9mm_Pitch1.27mm, symbol MC34063A
- RV2: footprint Potentiometers:Potentiometer_Bourns_3296Y_3-8Zoll_Angular_ScrewUp -> SMD_Packages:POT_SMD
Connections:
- net labels added: A1A, P34A, P35A, P36A, P38A, P40A
- wire segments 138 -> 114
Other:
- note added: "DC_driver\n"

Commit message: Update
Changed lines of the file:
@@
 P38A
 Text Label 1800 2950 0    60   ~ 0
-A1
+A1A
 Text Label 3050 2050 0    60   ~ 0
 P40A
